File: Hardware/PCBs/0x02.sch (EAGLE design)
At the start: 42 parts, among them IC1 78L05Z, IC2 TL072, IC3 4050N, SW1 TL2285

Commit message: Checkin of code & PCB for version 3 with DAC instead of PWM output.
Parts:
- removed IC3: 4050N, 40xx:4050N
- removed LED2: Red, led:LED5MM
- added Q1: 2N3906, transistor-pnp:2N3906
- added R14: 10k, rcl:R-EU_0207/2V
- added R17: 100k, rcl:R-EU_0207/2V
- added T1: 2N3904, transistor:2N3904
- added U$3: MCP4921, adafruit_mcp:MCP4921
- C8, C9: value 10n -> 470p
- R13: value 1k -> 100k
- R4: device rcl:R-EU_0207/7 -> rcl:R-EU_0207/2V
Connections:
- removed net GATE: IC3B.I, IC3C.O, IC3D.I, U$1.(PCINT8/XTAL1/CLKI)PB0
- removed net MISO: U$1.(PCINT5/OC1B/MISO/DO/ADC5)PA5, U$2.1
- removed net MOSI: U$1.(PCINT6/OC1A/SDA/MOSI/ADC6)PA6, U$2.4
- removed net N$17: IC3B.O, R15.1
- removed net N$18: IC3F.O, R16.1
- removed net N$20: LED2.C, R13.2
- removed net PWM_B: IC3A.I, IC3F.I, U$1.(PCINT7/ICP/OC0B/ADC7)PA7
- new net DAC_OUT: R3.1, U$3.DACA
- new net GATE_IN: R14.2, R17.2, T1.C, U$1.(PCINT8/XTAL1/CLKI)PB0
- new net GATE_OUT: R15.1, U$1.(PCINT7/ICP/OC0B/ADC7)PA7
- new net MISO_DO: U$1.(PCINT5/OC1B/MISO/DO/ADC5)PA5, U$2.1, U$3.SDI
- new net MOSI_SS: U$1.(PCINT6/OC1A/SDA/MOSI/ADC6)PA6, U$2.4, U$3.#CS
- new net N$4: Q1.B, R17.1
- net +5V: now also Q1.E, R14.1, U$3.REFA, U$3.VDD; no longer IC3P.VDD, LED2.A
- net GND: now also T1.E, U$3.AVSS, U$3.LDAC; no longer IC3E.I, IC3P.VSS
- net N$1: now also T1.B; no longer IC3A.O
- net N$2: now also Q1.C; no longer IC3D.O
- net N$8: now also R13.2; no longer IC3C.I
- net PWM_A: now also R16.1; no longer R3.1
- net SCK: now also U$3.SCK
Other:
- note added: "CV level Indicator LED"
- note added: "GATE Indicator LED"
- moved on the sheet: C2, GATE_IN, GATE_THRU, LED1, LED3, R13, R15, R16, R5

Commit message: Added jumper to set voltage output range, -5V to +5V or 0-+10V.
Parts:
- added JP2: (no value), pinhead:PINHD-1X3
Connections:
- new net N$6: JP2.2, R2.1
- net +5V: now also JP2.1; no longer R2.1
- net GND: now also JP2.3
Other:
- note added: "Voltage range jumper To +5V: Bipolar -5 to +5V output To GND: Unipolar 0 to +10V output"
Changed lines of the file:
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@@
 <grid distance="0.1" unitdist="inch" unit="inch" style="lines" multiple="1" display="no" altdistance="0.01" altunitdist="inch" altunit="inch"/>
 <layers>
-<layer number="1" name="Top" color="4" fill="1" visible="yes" active="no"/>
-<layer number="16" name="Bottom" color="1" fill="1" visible="yes" active="no"/>
-<layer number="17" name="Pads" color="2" fill="1" visible="yes" active="no"/>
-<layer number="18" name="Vias" color="2" fill="1" visible="yes" active="no"/>
-<layer number="19" name="Unrouted" color="6" fill="1" visible="yes" active="no"/>
-<layer number="20" name="Dimension" color="15" fill="1" visible="yes" active="no"/>
-<layer number="21" name="tPlace" color="7" fill="1" visible="yes" active="no"/>
-<layer number="22" name="bPlace" color="7" fill="1" visible="yes" active="no"/>
-<layer number="23" name="tOrigins" color="15" fill="1" visible="yes" active="no"/>
-<layer number="24" name="bOrigins" color="15" fill="1" visible="yes" active="no"/>
-<layer number="25" name="tNames" color="7" fill="1" visible="yes" active="no"/>
-<layer number="26" name="bNames" color="7" fill="1" visible="yes" active="no"/>
-<layer number="27" name="tValues" color="7" fill="1" visible="yes" active="no"/>
-<layer number="28" name="bValues" color="7" fill="1" visible="yes" active="no"/>
+<layer number="1" name="Top" color="4" fill="1" visible="no" active="no"/>
+<layer number="16" name="Bottom" color="1" fill="1" visible="no" active="no"/>
+<layer number="17" name="Pads" color="2" fill="1" visible="no" active="no"/>
+<layer number="18" name="Vias" color="2" fill="1" visible="no" active="no"/>
+<layer number="19" name="Unrouted" color="6" fill="1" visible="no" active="no"/>
+<layer number="20" name="Dimension" color="15" fill="1" visible="no" active="no"/>
+<layer number="21" name="tPlace" color="7" fill="1" visible="no" active="no"/>
+<layer number="22" name="bPlace" color="7" fill="1" visible="no" active="no"/>
+<layer number="23" name="tOrigins" color="15" fill="1" visible="no" active="no"/>
+<layer number="24" name="bOrigins" color="15" fill="1" visible="no" active="no"/>
+<layer number="25" name="tNames" color="7" fill="1" visible="no" active="no"/>
+<layer number="26" name="bNames" color="7" fill="1" visible="no" active="no"/>
+<layer number="27" name="tValues" color="7" fill="1" visible="no" active="no"/>
+<layer number="28" name="bValues" color="7" fill="1" visible="no" active="no"/>
 <layer number="29" name="tStop" color="7" fill="3" visible="no" active="no"/>
 <layer number="30" name="bStop" color="7" fill="6" visible="no" active="no"/>
@@
 <layer number="35" name="tGlue" color="7" fill="4" visible="no" active="no"/>
 <layer number="36" name="bGlue" color="7" fill="5" visible="no" active="no"/>
-<layer number="37" name="tTest" color="7" fill="1" visible="yes" active="no"/>
-<layer number="38" name="bTest" color="7" fill="1" visible="yes" active="no"/>
+<layer number="37" name="tTest" color="7" fill="1" visible="no" active="no"/>
+<layer number="38" name="bTest" color="7" fill="1" visible="no" active="no"/>
 <layer number="39" name="tKeepout" color="4" fill="11" visible="no" active="no"/>
 <layer number="40" name="bKeepout" color="1" fill="11" visible="no" active="no"/>
@@
 <layer number="44" name="Drills" color="7" fill="1" visible="no" active="no"/>
 <layer number="45" name="Holes" color="7" fill="1" visible="no" active="no"/>
-<layer number="46" name="Milling" color="3" fill="1" visible="yes" active="no"/>
-<layer number="47" name="Measures" color="7" fill="1" visible="yes" active="no"/>
-<layer number="48" name="Document" color="7" fill="1" visible="yes" active="no"/>
-<layer number="49" name="Reference" color="7" fill="1" visible="yes" active="no"/>
-<layer number="50" name="dxf" color="7" fill="1" visible="yes" active="no"/>
-<layer number="51" name="tDocu" color="7" fill="1" visible="yes" active="no"/>
-<layer number="52" name="bDocu" color="7" fill="1" visible="yes" active="no"/>
-<layer number="53" name="tGND_GNDA" color="7" fill="9" visible="yes" active="no"/>
-<layer number="54" name="bGND_GNDA" color="1" fill="9" visible="yes" active="no"/>
-<layer number="56" name="wert" color="7" fill="1" visible="yes" active="no"/>
+<layer number="46" name="Milling" color="3" fill="1" visible="no" active="no"/>
+<layer number="47" name="Measures" color="7" fill="1" visible="no" active="no"/>
+<layer number="48" name="Document" color="7" fill="1" visible="no" active="no"/>
+<layer number="49" name="Reference" color="7" fill="1" visible="no" active="no"/>
+<layer number="50" name="dxf" color="7" fill="1" visible="no" active="no"/>
+<layer number="51" name="tDocu" color="7" fill="1" visible="no" active="no"/>
+<layer number="52" name="bDocu" color="7" fill="1" visible="no" active="no"/>
+<layer number="53" name="tGND_GNDA" color="7" fill="9" visible="no" active="no"/>
+<layer number="54" name="bGND_GNDA" color="1" fill="9" visible="no" active="no"/>
+<layer number="56" name="wert" color="7" fill="1" visible="no" active="no"/>
 <layer number="90" name="Modules" color="5" fill="1" visible="yes" active="yes"/>
 <layer number="91" name="Nets" color="2" fill="1" visible="yes" active="yes"/>
 <layer number="92" name="Busses" color="1" fill="1" visible="yes" active="yes"/>
-<layer number="93" name="Pins" color="2" fill="1" visible="no" active="yes"/>
+<layer number="93" name="Pins" color="2" fill="1" visible="yes" active="yes"/>
 <layer number="94" name="Symbols" color="4" fill="1" visible="yes" active="yes"/>
 <layer number="95" name="Names" color="7" fill="1" visible="yes" active="yes"/>
@@
 <part name="GND8" library="supply1" deviceset="GND" device=""/>
 <part name="GND9" library="supply1" deviceset="GND" device=""/>
-<part name="P+4" library="supply1" deviceset="+5V" device=""/>
 <part name="P+6" library="supply1" deviceset="+12V" device=""/>
 <part name="P-3" library="supply1" deviceset="-12V" device=""/>
@@
 <part name="C2" library="rcl" deviceset="C-EU" device="025-025X050" value="100n"/>
 <part name="GND17" library="supply1" deviceset="GND" device=""/>
+<part name="JP2" library="pinhead" deviceset="PINHD-1X3" device=""/>
+<part name="P+4" library="supply1" deviceset="+5V" device=""/>
+<part name="GND18" library="supply1" deviceset="GND" device=""/>
 </parts>
 <sheets>
@@
 <text x="320.04" y="63.5" size="1.778" layer="91">CV level Indicator LED</text>
 <text x="320.04" y="91.44" size="1.778" layer="91">GATE Indicator LED</text>
+<text x="241.3" y="162.56" size="1.778" layer="91">Voltage range jumper
+To +5V: Bipolar -5 to +5V output
+To GND: Unipolar 0 to +10V output</text>
 </plain>
 <instances>
@@
 <instance part="GND8" gate="1" x="246.38" y="223.52" rot="R90"/>
 <instance part="GND9" gate="1" x="314.96" y="180.34"/>
-<instance part="P+4" gate="1" x="218.44" y="165.1" rot="R180"/>
 <instance part="P+6" gate="1" x="76.2" y="58.42"/>
 <instance part="P-3" gate="1" x="76.2" y="17.78"/>
@@
 <instance part="C2" gate="G$1" x="185.42" y="139.7"/>
 <instance part="GND17" gate="1" x="185.42" y="132.08"/>
+<instance part="JP2" gate="A" x="233.68" y="165.1"/>
+<instance part="P+4" gate="1" x="238.76" y="175.26"/>
+<instance part="GND18" gate="1" x="238.76" y="154.94"/>
 </instances>
 <busses>
@@
 <pinref part="GND17" gate="1" pin="GND"/>
 </segment>
+<segment>
+<pinref part="JP2" gate="A" pin="3"/>
+<wire x1="231.14" y1="162.56" x2="238.76" y2="162.56" width="0.1524" layer="91"/>
+<wire x1="238.76" y1="162.56" x2="238.76" y2="157.48" width="0.1524" layer="91"/>
+<pinref part="GND18" gate="1" pin="GND"/>
+</segment>
 </net>
 <net name="+5V" class="0">
@@
 <pinref part="P+3" gate="1" pin="+5V"/>
 <wire x1="210.82" y1="78.74" x2="210.82" y2="83.82" width="0.1524" layer="91"/>
-</segment>
-<segment>
-<pinref part="R2" gate="G$1" pin="1"/>
-<wire x1="218.44" y1="172.72" x2="218.44" y2="167.64" width="0.1524" layer="91"/>
-<pinref part="P+4" gate="1" pin="+5V"/>
 </segment>
 <segment>
@@
 <wire x1="292.1" y1="101.6" x2="292.1" y2="93.98" width="0.1524" layer="91"/>
 </segment>
+<segment>
+<pinref part="JP2" gate="A" pin="1"/>
+<wire x1="231.14" y1="167.64" x2="238.76" y2="167.64" width="0.1524" layer="91"/>
+<wire x1="238.76" y1="167.64" x2="238.76" y2="172.72" width="0.1524" layer="91"/>
+<pinref part="P+4" gate="1" pin="+5V"/>
+</segment>
 </net>
 <net name="MISO_DO" class="0">
@@
 </segment>
 </net>
+<net name="N$6" class="0">
+<segment>
+<pinref part="R2" gate="G$1" pin="1"/>
+<wire x1="218.44" y1="172.72" x2="218.44" y2="165.1" width="0.1524" layer="91"/>
+<pinref part="JP2" gate="A" pin="2"/>
+<wire x1="218.44" y1="165.1" x2="231.14" y2="165.1" width="0.1524" layer="91"/>
+</segment>
+</net>
 </nets>
 </sheet>
@@
 </schematic>
 </drawing>
+<compatibility>
+<note version="6.3" minversion="6.2.2" severity="warning">
+Since Version 6.2.2 text objects can contain more than one line,
+which will not be processed correctly with this version.
+</note>
+</compatibility>
 </eagle>

Commit message: Make voltage mixer into a true voltage adder (ext cv in tied to GND when unused, and 2x gain in output amp).
Parts:
- added R18, R19: 100k, rcl:R-EU_0207/2V
Connections:
- new net N$13: IC2B.-IN, R18.1, R19.2
- net GND: now also CV1IN.NORM, R19.1
- net N$15: now also R18.2; no longer IC2B.-IN
Changed lines of the file:
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@@
 <part name="P+4" library="supply1" deviceset="+5V" device=""/>
 <part name="GND18" library="supply1" deviceset="GND" device=""/>
+<part name="R18" library="rcl" deviceset="R-EU_" device="0207/2V" value="100k"/>
+<part name="R19" library="rcl" deviceset="R-EU_" device="0207/2V" value="100k"/>
+<part name="GND19" library="supply1" deviceset="GND" device=""/>
 </parts>
 <sheets>
@@
 <text x="320.04" y="63.5" size="1.778" layer="91">CV level Indicator LED</text>
 <text x="320.04" y="91.44" size="1.778" layer="91">GATE Indicator LED</text>
-<text x="241.3" y="162.56" size="1.778" layer="91">Voltage range jumper
+<text x="243.84" y="152.4" size="1.778" layer="91">Voltage range jumper
 To +5V: Bipolar -5 to +5V output
 To GND: Unipolar 0 to +10V output</text>
@@
 <instance part="P+4" gate="1" x="238.76" y="175.26"/>
 <instance part="GND18" gate="1" x="238.76" y="154.94"/>
+<instance part="R18" gate="G$1" x="279.4" y="182.88"/>
+<instance part="R19" gate="G$1" x="269.24" y="175.26" rot="R90"/>
+<instance part="GND19" gate="1" x="269.24" y="165.1"/>
 </instances>
 <busses>
@@
 <segment>
 <pinref part="CV1IN" gate="G$1" pin="RING"/>
-<wire x1="236.22" y1="223.52" x2="243.84" y2="223.52" width="0.1524" layer="91"/>
+<wire x1="236.22" y1="223.52" x2="238.76" y2="223.52" width="0.1524" layer="91"/>
 <pinref part="GND8" gate="1" pin="GND"/>
+<pinref part="CV1IN" gate="G$1" pin="NORM"/>
+<wire x1="238.76" y1="223.52" x2="243.84" y2="223.52" width="0.1524" layer="91"/>
+<wire x1="236.22" y1="220.98" x2="238.76" y2="220.98" width="0.1524" layer="91"/>
+<wire x1="238.76" y1="220.98" x2="238.76" y2="223.52" width="0.1524" layer="91"/>
+<junction x="238.76" y="223.52"/>
 </segment>
 <segment>
@@
 <pinref part="GND18" gate="1" pin="GND"/>
 </segment>
+<segment>
+<pinref part="R19" gate="G$1" pin="1"/>
+<pinref part="GND19" gate="1" pin="GND"/>
+<wire x1="269.24" y1="170.18" x2="269.24" y2="167.64" width="0.1524" layer="91"/>
+</segment>
 </net>
 <net name="+5V" class="0">
@@
 <pinref part="R7" gate="G$1" pin="1"/>
 <wire x1="287.02" y1="195.58" x2="289.56" y2="195.58" width="0.1524" layer="91"/>
-<pinref part="IC2" gate="B" pin="-IN"/>
 <wire x1="289.56" y1="195.58" x2="297.18" y2="195.58" width="0.1524" layer="91"/>
-<wire x1="271.78" y1="193.04" x2="269.24" y2="193.04" width="0.1524" layer="91"/>
-<wire x1="269.24" y1="193.04" x2="269.24" y2="187.96" width="0.1524" layer="91"/>
-<wire x1="269.24" y1="187.96" x2="289.56" y2="187.96" width="0.1524" layer="91"/>
-<wire x1="289.56" y1="187.96" x2="289.56" y2="195.58" width="0.1524" layer="91"/>
+<wire x1="289.56" y1="182.88" x2="289.56" y2="195.58" width="0.1524" layer="91"/>
 <junction x="289.56" y="195.58"/>
+<pinref part="R18" gate="G$1" pin="2"/>
+<wire x1="289.56" y1="182.88" x2="284.48" y2="182.88" width="0.1524" layer="91"/>
 </segment>
 </net>
@@
 </segment>
 </net>
+<net name="N$13" class="0">
+<segment>
+<pinref part="IC2" gate="B" pin="-IN"/>
+<wire x1="271.78" y1="193.04" x2="269.24" y2="193.04" width="0.1524" layer="91"/>
+<pinref part="R18" gate="G$1" pin="1"/>
+<wire x1="274.32" y1="182.88" x2="269.24" y2="182.88" width="0.1524" layer="91"/>
+<wire x1="269.24" y1="182.88" x2="269.24" y2="187.96" width="0.1524" layer="91"/>
+<pinref part="R19" gate="G$1" pin="2"/>
+<wire x1="269.24" y1="187.96" x2="269.24" y2="193.04" width="0.1524" layer="91"/>
+<wire x1="269.24" y1="182.88" x2="269.24" y2="180.34" width="0.1524" layer="91"/>
+<junction x="269.24" y="182.88"/>
+</segment>
+</net>
